File: BBB-Cape/KiCAD/Pins and Connectors.sch (KiCad schematic (older format))
At the start: 20 parts, among them J1 01x06_Stackable Header, P8 02x23_Stackable Header, P9 02x23_Stackable Header, SW1 W5500_RST, SW2 SYS_RST, SW3 Power

Commit message: BBB for review
Parts:
- removed I2C1_0: Conn_01x02, Pin_Headers:Pin_Header_Straight_1x02_Pitch2.54mm_SMD_Pin1Left, symbol Conn_01x02
- added I2C2_2: Conn_01x02, Pin_Headers:Pin_Header_Straight_1x02_Pitch2.54mm_SMD_Pin1Left, symbol Conn_01x02
- added P3, P4: 02x23_Stackable Header, Pin_Headers:Pin_Header_Straight_2x23_Pitch2.54mm, symbol Conn_02x23_Odd_Even
- renumbered I2C2_0 to I2C2_1, J1 to J9, P9 to P1, P8 to P2, R21 to R1
Connections:
- net +3V3: now also P4.3 (Pin_3), P4.4 (Pin_4)
- net +5V: now also P4.5 (Pin_5), P4.6 (Pin_6)
- net AIN0: now also P4.39 (Pin_39)
- net AIN1: now also P4.40 (Pin_40)
- net AIN2: now also P4.37 (Pin_37)
- net AIN3: now also P4.38 (Pin_38)
- net AIN4: now also P4.33 (Pin_33)
- net AIN5: now also P4.36 (Pin_36)
- net AIN6: now also P4.35 (Pin_35)
- net EHRPWM1A: now also P4.14 (Pin_14)
- net EHRPWM1B: now also P4.16 (Pin_16)
- net EHRPWM2A: now also P3.19 (Pin_19), P3.45 (Pin_45)
- net EHRPWM2B: now also P3.13 (Pin_13), P3.46 (Pin_46)
- net GND: now also P3.1 (Pin_1), P3.2 (Pin_2), P4.1 (Pin_1), P4.2 (Pin_2), P4.43 (Pin_43), P4.44 (Pin_44), P4.45 (Pin_45), P4.46 (Pin_46)
- net GNDA_ADC: now also P4.34 (Pin_34)
- net GPIO49: now also P4.23 (Pin_23)
- net GPIO_115: now also P4.27 (Pin_27)
- net GPIO_117: now also P4.25 (Pin_25)
- net GPIO_26: now also P3.14 (Pin_14)
- net GPIO_27: now also P3.17 (Pin_17)
- net GPIO_32: now also P3.25 (Pin_25)
- net GPIO_33: now also P3.24 (Pin_24)
- net GPIO_34: now also P3.5 (Pin_5)
- net GPIO_35: now also P3.6 (Pin_6)
- net GPIO_36: now also P3.23 (Pin_23)
- net GPIO_37: now also P3.22 (Pin_22)
- net GPIO_38: now also P3.3 (Pin_3)
- net GPIO_39: now also P3.4 (Pin_4)
- net GPIO_46: now also P3.16 (Pin_16)
- net GPIO_47: now also P3.15 (Pin_15)
- net GPIO_48: now also P4.15 (Pin_15)
- net GPIO_60: now also P4.12 (Pin_12)
- net GPIO_61: now also P3.26 (Pin_26)
- net GPIO_65: now also P3.18 (Pin_18)
- net I2C1_SCL/SPI0_CS0: now also P4.17 (Pin_17)
- net I2C1_SCL/UART1_TXD: now also P4.24 (Pin_24)
- net I2C1_SDA/SPI0_DI: now also P4.18 (Pin_18)
- net I2C1_SDA/UART1_RXD: now also P4.26 (Pin_26)
- net I2C2_SCL/SPI0_DO/UART2_TXD: now also I2C2_2.1 (Pin_1), P4.21 (Pin_21)
- net I2C2_SCL/SPI1_CS1/UART1_RTSn: now also P4.19 (Pin_19)
- net I2C2_SDA/SPI1_CS0/UART1_CTSn: now also P4.20 (Pin_20)
- net I2C2_SDA/SPIO_SCLK/UART2_RXD: now also I2C2_2.2 (Pin_2), P4.22 (Pin_22)
- net PRU0_14OUT: now also P3.12 (Pin_12)
- net PRU0_15OUT: now also P3.11 (Pin_11)
- net PRU1_10: now also P3.28 (Pin_28)
- net PRU1_11: now also P3.30 (Pin_30)
- net PRU1_12: now also P3.21 (Pin_21)
- net PRU1_13: now also P3.20 (Pin_20)
- net PRU1_2: now also P3.43 (Pin_43)
- net PRU1_3: now also P3.44 (Pin_44)
- net PRU1_4: now also P3.41 (Pin_41)
- net PRU1_5: now also P3.42 (Pin_42)
- net PRU1_6: now also P3.39 (Pin_39)
- net PRU1_7: now also P3.40 (Pin_40)
- net PRU1_8: now also P3.27 (Pin_27)
- net PRU1_9: now also P3.29 (Pin_29)
- net PWR_BUT: now also P4.9 (Pin_9)
- net SPI1_CS0: now also P4.28 (Pin_28)
- net SPI1_CS1/UART3_TXD: now also P4.42 (Pin_42)
- net SPI1_D0: now also P4.29 (Pin_29)
- net SPI1_DI: now also P4.30 (Pin_30)
- net SPI1_SCLK: now also P4.31 (Pin_31)
- net SYS_5V: now also P4.7 (Pin_7), P4.8 (Pin_8)
- net SYS_RESETn: now also P4.10 (Pin_10)
- net TIMER4: now also P3.7 (Pin_7)
- net TIMER5: now also P3.9 (Pin_9)
- net TIMER6: now also P3.10 (Pin_10)
- net TIMER7: now also P3.8 (Pin_8)
- net UART3_CTSn: now also P3.36 (Pin_36)
- net UART3_RTSn: now also P3.34 (Pin_34)
- net UART4_CTSn: now also P3.35 (Pin_35)
- net UART4_RTSn: now also P3.33 (Pin_33)
- net UART4_RXD: now also P4.11 (Pin_11)
- net UART4_TXD: now also P4.13 (Pin_13)
- net UART5_CTSn+: now also P3.31 (Pin_31)
- net UART5_RTSn: now also P3.32 (Pin_32)
- net UART5_RXD+: now also P3.38 (Pin_38)
- net UART5_TXD+: now also P3.37 (Pin_37)
- net VDD_ADC: now also P4.32 (Pin_32)
- net W5500_INT: now also P4.41 (Pin_41)
Other:
- moved on the sheet: D1, R1, SPI0_1, SPI1_1, SW1, SW2, SW3
