File: BBB-Cape/KiCAD/RJ45 and WIZnet W5500.sch (KiCad schematic (older format))
At the start: 41 parts, among them J2 RJ45-TRANSFO, U1 WIZnet W5500, Y1 25MHz

Commit message: BBB for review
Parts:
- L2: renamed from L1; value HH-1M1608-121JT -> BLM21PG121SN1D; footprint (none) -> Inductors_SMD:L_0805_HandSoldering
- renumbered C4 to C10, C1 to C11, C5 to C12, C2 to C13, C6 to C14, C7 to C15, C10 to C16, C11 to C17, C8 to C18, C9 to C19, C12 to C20, C13 to C21, C14 to C22, C15 to C23, C16 to C24, C17 to C25, C3 to C9, J2 to J11, R6 to R10, R7 to R11, R3 to R12, R8 to R13, R10 to R14, R11 to R15, R12 to R16, R13 to R17, R14 to R18, R15 to R19, R16 to R20, R17 to R21, R18 to R22, R9 to R23, R19 to R24, R20 to R25, R1 to R6, R4 to R7, R5 to R8, R2 to R9, U1 to U2
Connections:
- net SPI1_DO renamed SPI1_D0
